File: Circuit/robotrace_v2_Sidemarker/robotrace_v2_Sidemarker.kicad_pcb (KiCad board)
At the start: 2 copper layers, 42 x 7 mm, 9 parts, among them J2 Conn_01x03, U1 LBR-123F, U2 LBR-123F

Commit message: 回路図を最新版に更新
Parts:
- added JP1: Out, Jumper:SolderJumper-2_P1.3mm_Open_TrianglePad1.0x1.5mm, F.Cu at (165.9, 97.7)
- added JP2: In, Jumper:SolderJumper-2_P1.3mm_Open_TrianglePad1.0x1.5mm, F.Cu at (153.7, 97.6)
- moved R3 16.8 mm to (161.8, 99.0)
- moved U2 13.0 mm to (169.7, 98.2)
- moved R4 12.3 mm to (163.4, 99.0)
- moved C2 7.62 mm to (160.4, 98.9)
- moved C1 7.22 mm to (159.2, 98.9)
- moved R1 3.75 mm to (157.8, 99.0)
- moved R2 1.00 mm to (156.2, 99.0)
Connections:
- R2 pad 2: Net-(J2-Pin_2) -> Net-(JP2-A)
- R4 pad 2: Net-(J2-Pin_2) -> Net-(JP1-A)
- U1 pad 4: Net-(J2-Pin_2) -> Net-(JP2-A)
- U2 pad 4: Net-(J2-Pin_2) -> Net-(JP1-A)
Routing:
- net Net-(J2-Pin_2): track 47.6 -> 22.5 mm, vias 0 -> 1
- net +5V: track 36.9 -> 22.8 mm
- net Net-(JP2-A): track 0.00 -> 8.30 mm
- net GND2: track 64.7 -> 56.7 mm, vias 14 -> 2
- net Net-(JP1-A): track 0.00 -> 6.50 mm
- net Net-(U2-Anode): track 5.63 -> 10.7 mm
- net Net-(U1-Anode): track 3.83 -> 7.81 mm
Other:
- board size 42 x 7 mm -> 29 x 7 mm
