File: Circuit/robotrace_v2_Sidemarker/robotrace_v2_Sidemarker.kicad_sch (KiCad schematic)
At the start: 9 parts, among them J2 Conn_01x03, U1 LBR-123F, U2 LBR-123F

Commit message: 回路図を最新版に更新
Parts:
- added JP1: Out, Jumper:SolderJumper-2_P1.3mm_Open_TrianglePad1.0x1.5mm, symbol Jumper:Jumper_2_Open
- added JP2: In, Jumper:SolderJumper-2_P1.3mm_Open_TrianglePad1.0x1.5mm, symbol Jumper:Jumper_2_Open
Connections:
- new net: JP2.1 (A), R2.2, U1.4 (Collector)
- new net: J2.2 (Pin_2), JP1.2 (B), JP2.2 (B)
- new net: JP1.1 (A), R4.2, U2.4 (Collector)
Other:
- moved on the sheet: C1, C2, R1, R2, R3, R4, U1, U2
