File: Circuit/robotrace_v2_main_v2/robotrace_v2_main_v2.kicad_pcb (KiCad board)
At the start: 4 copper layers, 48 x 30 mm, 118 parts, among them J1 MOTOR1, J10 Sidemarker_L, J11 Sidemarker_R, J12 GPIO, J13 ST-Link, J2 BATT, J3 MOTOR1, J4 FFC, J5 Encoder1, J6 Encoder1, J7 FAN, J9 Micro_SD_Card, Q1 DMN1054UCB4, Q2 DMN1054UCB4, Q3 DMN1054UCB4, Q4 Q_NMOS_GSD, SW1 SW_SPDT_321, SW2 USER_SW_L, SW3 USER_SW_R, U1 STM32F446RETx, U10 SN74LVC1G18DCKR, U2 TPS63070, U3 ADM7172, U4 ENS7403, U7 U7, U9 SN74LVC1G18DCKR, Y1 ECS-2520S33-120-FN-TR

Commit message: 回路データとSTEPを更新
Parts:
- J1, J2, J3, J7: footprint Connector_Molex:Molex_SPOX_5267-02A_1x02_P2.50mm_Vertical -> robot_contest:Molex_mini-SPOX_1x02_P2.54mm_Horizontal
- moved J1 2.55 mm to (144.1, 81.5), turned to -90 degrees
- moved J3 2.55 mm to (184.3, 84.0), turned to 90 degrees
- moved J2 2.54 mm to (144.1, 89.9), turned to -90 degrees
- moved J7 2.50 mm to (184.3, 92.4), turned to 90 degrees
