File: Circuit/robotrace_v2_main_v2/robotrace_v2_main_v2.kicad_sch (KiCad schematic)
At the start: 118 parts, among them J1 MOTOR1, J10 Sidemarker_L, J11 Sidemarker_R, J12 GPIO, J13 ST-Link, J2 BATT, J3 MOTOR1, J4 FFC, J5 Encoder1, J6 Encoder1, J7 FAN, J9 Micro_SD_Card, Q1 DMN1054UCB4, Q2 DMN1054UCB4, Q3 DMN1054UCB4, Q4 Q_NMOS_GSD, SW1 SW_SPDT_321, SW2 USER_SW_L, SW3 USER_SW_R, U1 STM32F446RETx, U10 SN74LVC1G18DCKR, U2 TPS63070, U3 ADM7172, U4 ESN7403, U9 SN74LVC1G18DCKR, Y1 ECS-2520S33-120-FN-TR

Commit message: 回路データとSTEPを更新
Parts:
- J1, J2, J3, J7: footprint Connector_Molex:Molex_SPOX_5267-02A_1x02_P2.50mm_Vertical -> robot_contest:Molex_mini-SPOX_1x02_P2.54mm_Horizontal
Changed lines of the file:
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@@
 (kicad_sch
-	(version 20231120)
+	(version 20250114)
 	(generator "eeschema")
-	(generator_version "8.0")
+	(generator_version "9.0")
 	(paper "A3")
 	(junction
@@
 			)
 		)
-		(property "Footprint" "Connector_Molex:Molex_SPOX_5267-02A_1x02_P2.50mm_Vertical"
+		(property "Footprint" "robot_contest:Molex_mini-SPOX_1x02_P2.54mm_Horizontal"
 			(at 394.97 163.83 0)
 			(effects
@@
 			)
 		)
-		(property "Footprint" "Connector_Molex:Molex_SPOX_5267-02A_1x02_P2.50mm_Vertical"
+		(property "Footprint" "robot_contest:Molex_mini-SPOX_1x02_P2.54mm_Horizontal"
 			(at 234.95 101.6 0)
 			(effects
@@
 			)
 		)
-		(property "Footprint" "Connector_Molex:Molex_SPOX_5267-02A_1x02_P2.50mm_Vertical"
+		(property "Footprint" "robot_contest:Molex_mini-SPOX_1x02_P2.54mm_Horizontal"
 			(at 168.91 38.1 0)
 			(effects
@@
 			)
 		)
-		(property "Footprint" "Connector_Molex:Molex_SPOX_5267-02A_1x02_P2.50mm_Vertical"
+		(property "Footprint" "robot_contest:Molex_mini-SPOX_1x02_P2.54mm_Horizontal"
 			(at 396.24 99.06 0)
 			(effects
@@
 		)
 	)
+	(embedded_fonts no)
 )
